File: hardware/backpack/backpack.kicad_pcb (KiCad board)
At the start: 4 copper layers, 31.7 x 110 mm, 102 parts, among them J1 Conn_01x15, J2 Conn_02x06_Top_Bottom, J3 Conn_02x06_Top_Bottom, J4 AUDIO JACK PJ-324M0, J5 AUDIO JACK PJ-324M0, J6 CONN 2x5 P=2.54mm, J7 USB_C, J8 MICROMOD-2222, J9 USB_C, Q2 2N7002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

Commit message: updates before fab 04-04-24
Parts:
- C1, C10, C13, C14, C17, C2, C3, C4, C5, C6, C7, C8, C9: value 100nF/10V/20%/X5R/C0402 -> 0.1uF
- R1, R27: value 10k -> 10K
- R19, R20, R21, R22: value 5.1k -> 5.1K
- R25, R26, R6, R7: value 27R/R0402 -> 27R
- R29, R30, R5, R8: value 100R/R0402 -> 100R
- R3, R4: value 10k/R0402 -> 10K
- SW1, SW2: value ~ -> SW_Tactile_SPST
- U1: footprint Package_SO:SOP-8_3.9x4.9mm_P1.27mm -> Package_SO:SOIC-8W_5.3x5.3mm_P1.27mm
- moved C4 1.57 mm to (12.4, 21.4), turned to -90 degrees
- moved U1 0.68 mm to (8.69, 16.7)
- moved R8 0.30 mm to (6.31, 22.4)
- moved C3 0.19 mm to (12.2, 16.3)
Routing:
- net GND: track 61.4 -> 67.4 mm
- net /rp2040_jtag/IO3: track 11.5 -> 15.9 mm, vias 0 -> 2
- net /rp2040_jtag/CLK: track 13.9 -> 12.3 mm
- net /rp2040_jtag/IO0: track 12.0 -> 13.5 mm
- net ECP5_A3: track 74.9 -> 73.6 mm
- net /rp2040_jtag/IO2: track 10.2 -> 11.2 mm
- net +2V5: track 50.8 -> 49.9 mm
- net /rp2040_jtag/IO1: track 9.17 -> 9.73 mm
- net /rp2040_jtag/~{BOOTSEL}: track 5.40 -> 4.84 mm
- net ECP5_A7: track 78.4 -> 78.2 mm, vias 4 -> 6
