File: hardware/backpack/midi.kicad_sch (KiCad schematic)
At the start: 13 parts, among them J4 MIDI_TRS_A, J5 MIDI_TRS_A, Q2 2N7002, Q3 2N7002, U4 H11L1SR2M

Commit message: fix footprint errors and pin assignments on ffc
Parts:
- removed J4, J5: MIDI_TRS_A, pj3410:pj324m, symbol Connector_Audio:AudioJack2_Ground_SwitchT
- added J4, J5: AUDIO JACK PJ-324M0, pj3410:pj324m, symbol Connector:AudioJack2_Ground_Switch
Connections:
- net at D1.2 (A), U4.2: now also J4.T
- net at R14.1: now also J5.T
- net at R13.1: now also J5.S
- net at R10.1: now also J4.S
- no-connect marks 4 -> 6

Commit message: updates before fab 04-04-24
Parts:
- D1: lcsc# C2840959 -> C493190
- R10, R11, R16: lcsc# C112291 -> C25091
- R12: lcsc# C105871 -> C25900
- R13: lcsc# C138002 -> C25105
- R14: lcsc# C138066 -> C25077
- R15: lcsc# C2935237 -> C11702
Changed lines of the file:
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@@
 			)
 		)
-		(property "lcsc#" "C2840959"
+		(property "lcsc#" "C493190"
 			(at 143.51 69.85 0)
 			(effects
@@
 			)
 		)
-		(property "lcsc#" "C138066"
+		(property "lcsc#" " C25077"
 			(at 179.07 105.41 0)
 			(effects
@@
 			)
 		)
-		(property "lcsc#" "C105871"
+		(property "lcsc#" " C25900"
 			(at 148.59 104.14 0)
 			(effects
@@
 			)
 		)
-		(property "lcsc#" "C2935237"
+		(property "lcsc#" " C11702"
 			(at 185.42 64.77 0)
 			(effects
@@
 			)
 		)
-		(property "lcsc#" "C112291"
+		(property "lcsc#" " C25091"
 			(at 137.16 66.04 0)
 			(effects
@@
 			)
 		)
-		(property "lcsc#" "C112291"
+		(property "lcsc#" " C25091"
 			(at 137.16 113.03 0)
 			(effects
@@
 			)
 		)
-		(property "lcsc#" "C112291"
+		(property "lcsc#" " C25091"
 			(at 191.77 69.85 0)
 			(effects
@@
 			)
 		)
-		(property "lcsc#" "C138002"
+		(property "lcsc#" "C25105"
 			(at 179.07 102.87 0)
 			(effects
