File: hardware/panel/eurorack-pmod-panel.kicad_pcb (KiCad board)
At the start: 2 copper layers, 30 x 128.5 mm, 12 parts

Commit message: fab panel proto2
Parts:
- added G***: LOGO, LOGO, F.Cu at (26.8, 7.50)
