File: hardware/tiliqua-motherboard/midi.kicad_sch (KiCad schematic)
At the start: 13 parts, among them J4 AUDIO JACK PJ-324M0, J5 AUDIO JACK PJ-324M0, Q2 2N7002, Q3 2N7002, U4 H11L1SR2M

Commit message: hardware/r2: squash in all changes for tiliqua R2 (#17)
* squash in all changes for Tiliqua R2
* add schematics for all components of Tiliqua R2
* update README and add lightbox photos
Parts:
- removed J5: AUDIO JACK PJ-324M0, pj3410:pj324m, symbol Connector:AudioJack2_Ground_Switch
- removed Q2, Q3: 2N7002, Package_TO_SOT_SMD:SOT-23, symbol Transistor_FET:2N7002
- removed R11: 220R, Resistor_SMD:R_0402_1005Metric, symbol Device:R
- removed R12: 4K7, Resistor_SMD:R_0402_1005Metric, symbol Device:R
- removed R13: 33R, Resistor_SMD:R_0402_1005Metric, symbol Device:R
- removed R14: 10R, Resistor_SMD:R_0402_1005Metric, symbol Device:R
- J4: value AUDIO JACK PJ-324M0 -> ~; footprint pj3410:pj324m -> jacks:AUDIO-TH_PJ-325M; lcsc# C2884986 -> C2884942; mfg# PJ-324M0 -> (none)
- R10, R16: lcsc# C25091 -> C25091
Connections:
- net GND: now also J4.G
- no-connect marks 6 -> 2
Other:
- note added: "TODO: PTH through panel for shielding"
