File: hardware/tiliqua-motherboard/midi.kicad_sch (KiCad schematic)
At the start: 13 parts, among them J4 AUDIO JACK PJ-324M0, J5 AUDIO JACK PJ-324M0, Q2 2N7002, Q3 2N7002, U4 H11L1SR2M

Commit message: final 90deg USB and button model
Connections:
- net GND: now also J4.G, J5.G
- no-connect marks 6 -> 4
Other:
- note added: "TODO: PTH through panel for shielding"
Changed lines of the file:
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@@
-	)
-	(no_connect
-		(at 116.84 78.74)
-	)
-	(no_connect
-		(at 190.5 115.57)
 	)
 	(no_connect
@@
 		)
 	)
+	(polyline
+		(pts
+			(xy 111.76 83.185) (xy 114.935 83.185)
+		)
+		(stroke
+			(width 0)
+			(type default)
+		)
+	)
 	(wire
 		(pts
@@
 		)
 	)
+	(polyline
+		(pts
+			(xy 111.76 87.63) (xy 111.76 83.185)
+		)
+		(stroke
+			(width 0)
+			(type default)
+		)
+	)
 	(wire
 		(pts
@@
 	(wire
 		(pts
+			(xy 190.5 120.65) (xy 190.5 115.57)
+		)
+		(stroke
+			(width 0)
+			(type default)
+		)
+	)
+	(wire
+		(pts
 			(xy 156.21 107.95) (xy 148.59 107.95)
 		)
@@
 	(wire
 		(pts
+			(xy 116.84 81.28) (xy 116.84 78.74)
+		)
+		(stroke
+			(width 0)
+			(type default)
+		)
+	)
+	(wire
+		(pts
 			(xy 133.35 113.03) (xy 128.27 113.03)
 		)
@@
 			(width 0)
 			(type default)
+		)
+	)
+	(text "TODO: PTH through panel for shielding"
+		(exclude_from_sim no)
+		(at 115.824 89.916 0)
+		(effects
+			(font
+				(size 1.27 1.27)
+			)
 		)
 	)
@@
 					(unit 1)
 				)
+			)
+		)
+	)
+	(symbol
+		(lib_id "power:GND")
+		(at 190.5 120.65 0)
+		(mirror y)
+		(unit 1)
+		(exclude_from_sim no)
+		(in_bom yes)
+		(on_board yes)
+		(dnp no)
+		(fields_autoplaced yes)
+		(property "Reference" "#PWR074"
+			(at 190.5 127 0)
+			(effects
+				(font
+					(size 1.27 1.27)
+				)
+				(hide yes)
+			)
+		)
+		(property "Value" "GND"
+			(at 190.5 125.73 0)
+			(effects
+				(font
+					(size 1.27 1.27)
+				)
+			)
+		)
+		(property "Footprint" ""
+			(at 190.5 120.65 0)
+			(effects
+				(font
+					(size 1.27 1.27)
+				)
+				(hide yes)
+			)
+		)
+		(property "Datasheet" ""
+			(at 190.5 120.65 0)
+			(effects
+				(font
+					(size 1.27 1.27)
+				)
+				(hide yes)
+			)
+		)
+		(property "Description" ""
+			(at 190.5 120.65 0)
+			(effects
+				(font
+					(size 1.27 1.27)
+				)
+				(hide yes)
+			)
+		)
+		(pin "1"
+		)
+		(instances
+			(project "tiliqua-motherboard"
+				(path "/df6062c3-a570-4505-924c-c7fe32df3670/dd79b704-4c8d-4498-8ec1-0bb3e9e805ab"
+					(reference "#PWR074")
+					(unit 1)
+				)
+			)
+		)
+	)
+	(symbol
+		(lib_id "power:GND")
+		(at 116.84 81.28 0)
+		(mirror y)
+		(unit 1)
+		(exclude_from_sim no)
+		(in_bom yes)
+		(on_board yes)
+		(dnp no)
+		(fields_autoplaced yes)
+		(property "Reference" "#PWR075"
+			(at 116.84 87.63 0)
+			(effects
+				(font
+					(size 1.27 1.27)
+				)
+				(hide yes)
+			)
+		)
+		(property "Value" "GND"
+			(at 116.84 86.36 0)
+			(effects
+				(font
+					(size 1.27 1.27)
+				)
+			)
+		)
+		(property "Footprint" ""
+			(at 116.84 81.28 0)
+			(effects
+				(font
+					(size 1.27 1.27)
+				)
+				(hide yes)
+			)
+		)
+		(property "Datasheet" ""
+			(at 116.84 81.28 0)
+			(effects
+				(font
+					(size 1.27 1.27)
+				)
+				(hide yes)
+			)
+		)
+		(property "Description" ""
+			(at 116.84 81.28 0)
+			(effects
+				(font
+					(size 1.27 1.27)
+				)
+				(hide yes)
+			)
+		)
+		(pin "1"
+		)
+		(instances
+			(project "tiliqua-motherboard"
+				(path "/df6062c3-a570-4505-924c-c7fe32df3670/dd79b704-4c8d-4498-8ec1-0bb3e9e805ab"
+					(reference "#PWR075")
+					(unit 1)
+				)

Commit message: pj325 for midi
Parts:
- J4: value AUDIO JACK PJ-324M0 -> (none); footprint pj3410:pj324m -> jacks:AUDIO-TH_PJ-325M; lcsc# C2884986 -> (none); mfg# PJ-324M0 -> (none)
- J5: footprint pj3410:pj324m -> jacks:AUDIO-TH_PJ-325M; lcsc# C2884986 -> (none); mfg# PJ-324M0 -> (none)
Changed lines of the file:
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@@
 			)
 		)
-		(property "Footprint" "pj3410:pj324m"
+		(property "Footprint" "jacks:AUDIO-TH_PJ-325M"
 			(at 190.5 102.87 0)
 			(effects
@@
 			)
 		)
-		(property "Datasheet" "https://datasheet.lcsc.com/lcsc/2110120730_XKB-Connectivity-PJ-324M0_C2884986.pdf"
+		(property "Datasheet" ""
 			(at 190.5 102.87 0)
 			(effects
@@
 			)
 		)
-		(property "lcsc#" "C2884986"
+		(property "lcsc#" ""
 			(at 190.5 107.95 0)
 			(effects
@@
 			)
 		)
-		(property "mfg#" "PJ-324M0"
+		(property "mfg#" ""
 			(at 190.5 107.95 0)
 			(effects
@@
 			)
 		)
-		(property "Value" "AUDIO JACK PJ-324M0"
+		(property "Value" ""
 			(at 116.205 61.595 0)
 			(effects
@@
 			)
 		)
-		(property "Footprint" "pj3410:pj324m"
+		(property "Footprint" "jacks:AUDIO-TH_PJ-325M"
 			(at 116.84 66.04 0)
 			(effects
@@
 			)
 		)
-		(property "Datasheet" "https://datasheet.lcsc.com/lcsc/2110120730_XKB-Connectivity-PJ-324M0_C2884986.pdf"
+		(property "Datasheet" ""
 			(at 116.84 66.04 0)
 			(effects
@@
 			)
 		)
-		(property "lcsc#" "C2884986"
+		(property "lcsc#" ""
 			(at 116.84 71.12 0)
 			(effects
@@
 			)
 		)
-		(property "mfg#" "PJ-324M0"
+		(property "mfg#" ""
 			(at 116.84 71.12 0)
 			(effects

Commit message: big HDMI
Parts:
- removed J5: AUDIO JACK PJ-324M0, jacks:AUDIO-TH_PJ-325M, symbol Connector:AudioJack2_Ground_Switch
- removed Q2, Q3: 2N7002, Package_TO_SOT_SMD:SOT-23, symbol Transistor_FET:2N7002
- removed R11: 220R, Resistor_SMD:R_0402_1005Metric, symbol Device:R
- removed R12: 4K7, Resistor_SMD:R_0402_1005Metric, symbol Device:R
- removed R13: 33R, Resistor_SMD:R_0402_1005Metric, symbol Device:R
- removed R14: 10R, Resistor_SMD:R_0402_1005Metric, symbol Device:R
- J4: value (none) -> ~
Connections:
- no-connect marks 4 -> 2

Commit message: add some part numbers
Parts:
- J4: lcsc# (none) -> C2884942
- R10, R16: lcsc# C25091 -> C25091
Changed lines of the file:
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@@
+			)
+		)
+		(property "Tol" ""
+			(at 143.51 69.85 0)
+			(effects
+				(font
+					(size 1.27 1.27)
+				)
+				(hide yes)
 			)
 		)
@@
 			)
 		)
+		(property "Tol" ""
+			(at 185.42 64.77 0)
+			(effects
+				(font
+					(size 1.27 1.27)
+				)
+				(hide yes)
+			)
+		)
 		(pin "1"
 		)
@@
 			)
 		)
-		(property "lcsc#" " C25091"
+		(property "lcsc#" "C25091"
+			(at 137.16 66.04 0)
+			(effects
+				(font
+					(size 1.27 1.27)
+				)
+				(hide yes)
+			)
+		)
+		(property "Tol" ""
 			(at 137.16 66.04 0)
 			(effects
@@
 		)
 		(property "lcsc#" "C20082"
+			(at 163.83 69.85 0)
+			(effects
+				(font
+					(size 1.27 1.27)
+				)
+				(hide yes)
+			)
+		)
+		(property "Tol" ""
 			(at 163.83 69.85 0)
 			(effects
@@
 			)
 		)
-		(property "lcsc#" " C25091"
+		(property "lcsc#" "C25091"
+			(at 191.77 69.85 0)
+			(effects
+				(font
+					(size 1.27 1.27)
+				)
+				(hide yes)
+			)
+		)
+		(property "Tol" ""
 			(at 191.77 69.85 0)
 			(effects
@@
 			)
 		)
-		(property "lcsc#" ""
+		(property "lcsc#" "C2884942 "
 			(at 116.84 71.12 0)
 			(effects
@@
 			(at 116.84 71.12 0)
 			(effects
+				(font
+					(size 1.27 1.27)
+				)
+				(hide yes)
+			)
+		)
+		(property "Tol" ""
+			(at 116.84 71.12 0)
+			(effects

Commit message: hw/mobo-r3: add LCSC database / associations
Parts:
- D1: LCSC (none) -> C493190
- J4: LCSC (none) -> C2884942
- R10, R16: LCSC (none) -> C25091
- R15: LCSC (none) -> C11702
- U4: LCSC (none) -> C20082
Changed lines of the file:
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@@
+			)
+		)
+		(property "LCSC" "C493190"
+			(at 146.05 69.85 0)
+			(effects
+				(font
+					(size 1.27 1.27)
+				)
+				(hide yes)
 			)
 		)
@@
 			)
 		)
+		(property "LCSC" "C11702"
+			(at 182.88 64.77 0)
+			(effects
+				(font
+					(size 1.27 1.27)
+				)
+				(hide yes)
+			)
+		)
 		(pin "1"
 		)
@@
 			)
 		)
+		(property "LCSC" "C25091"
+			(at 137.16 63.5 0)
+			(effects
+				(font
+					(size 1.27 1.27)
+				)
+				(hide yes)
+			)
+		)
 		(pin "1"
 		)
@@
 		(property "Tol" ""
 			(at 163.83 69.85 0)
+			(effects
+				(font
+					(size 1.27 1.27)
+				)
+				(hide yes)
+			)
+		)
+		(property "LCSC" "C20082"
+			(at 175.26 63.5 0)
 			(effects
 				(font
@@
 			)
 		)
+		(property "LCSC" "C25091"
+			(at 191.77 72.39 0)
+			(effects
+				(font
+					(size 1.27 1.27)
+				)
+				(hide yes)
+			)
+		)
 		(pin "1"
 		)
@@
 			(effects
 				(font
+					(size 1.27 1.27)
+				)
+				(hide yes)
+			)
+		)
+		(property "LCSC" "C2884942"
+			(at 116.205 59.055 0)
+			(effects
+				(font
