File: hardware/tiliqua-motherboard/power.kicad_sch (KiCad schematic)
At the start: 33 parts, among them J6 CONN 2x5 P=2.54mm, U10 TPS7A91, U5 AP63200WU

Commit message: hw/mobo-r3: add LCSC database / associations
Parts:
- C17, C25, C28, C30: LCSC (none) -> C307331
- C18: LCSC (none) -> C15195
- C19, C20, C23, C29, C32, C38: LCSC (none) -> C12891
- C21, C33: LCSC (none) -> C88795
- C31: LCSC (none) -> C77177
- C34: LCSC (none) -> C14663
- D2, D3: LCSC (none) -> C493190
- F1: LCSC (none) -> C883107
- F2: LCSC (none) -> C883103
- J6: LCSC (none) -> C492433
- L1, L2, L4, L5, L6, L7: LCSC (none) -> C14709
- L3: LCSC (none) -> C844996
- R17: LCSC (none) -> C861679
- R18: LCSC (none) -> C25776
- R42: LCSC (none) -> C29401
- R43: LCSC (none) -> C270609
- U10: LCSC (none) -> C2878140
- U5: LCSC (none) -> C2071868
